File: generalPassiveEEG/genPassiveEEG/genPassiveEEG.kicad_pcb (KiCad board)
At the start: 2 copper layers, 66 x 33 mm, 11 parts, among them J1 ToAmp, J10 Ch 5, J12 GND, J2 Ch 7, J3 Ch 1, J4 Ch 3, J5 Ch 8, J6 REF, J7 Ch 4, J8 Ch 6, J9 Ch 2

Commit message: revised both PCBs and added drill holes to genPassiveEEG
Other:
- board size 66 x 33 mm -> 66 x 38.1 mm
Changed lines of the file:
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@@
 	)
 	(gr_line
-		(start 94 50)
-		(end 28 50)
+		(start 94.05 44.85)
+		(end 28 44.85)
 		(stroke
 			(width 0.05)
@@
 		(layer "Edge.Cuts")
 	)
+	(gr_circle
+		(center 41.09 49.24)
+		(end 43.32 51.08)
+		(stroke
+			(width 0.2)
+			(type solid)
+		)
+		(fill no)
+		(layer "Edge.Cuts")
+	)
+	(gr_circle
+		(center 88.888893 77.77)
+		(end 91.118893 79.61)
+		(stroke
+			(width 0.2)
+			(type solid)
+		)
+		(fill no)
+		(layer "Edge.Cuts")
+	)
+	(gr_circle
+		(center 80.75 48.86)
+		(end 82.98 50.7)
+		(stroke
+			(width 0.2)
+			(type solid)
+		)
+		(fill no)
+		(layer "Edge.Cuts")
+	)
 	(gr_line
-		(start 28 50)
+		(start 28 44.85)
 		(end 28 83)
 		(stroke
@@
 	(gr_line
 		(start 94 83)
-		(end 94 50)
+		(end 94.05 44.85)
 		(stroke
 			(width 0.05)
@@
 		(layer "Edge.Cuts")
 	)
+	(gr_circle
+		(center 33.088893 77.92)
+		(end 35.318893 79.76)
+		(stroke
+			(width 0.2)
+			(type solid)
+		)
+		(fill no)
+		(layer "Edge.Cuts")
+	)
